Commit message: take into account mode into urdf description

File: romea_rtls_transceiver_description/urdf/anchor.xacro (robot description, xacro)
@@ -1,9 +1,10 @@
 <?xml version="1.0"?>
 <robot name="anchor" xmlns:xacro="http://www.ros.org/wiki/xacro">
-  <xacro:macro name="anchor" params="name type conf id pan_id">
+  <xacro:macro name="anchor" params="mode name type conf id pan_id">
     <xacro:include filename="$(find romea_rtls_transceiver_description)/urdf/transceiver.xacro" />
     <link name="support" />
-    <xacro:transceiver prefix="" name="${name}" type="${type}" conf="${conf}" id=" ${id}"
-      pan_id=" ${id}" mode="standalone" parent_link="support" xyz=" 0.0 0.0 0.0" ros_namespace="" />
+    <xacro:transceiver prefix="" mode="${mode}" name="${name}" type="${type}" conf="${conf}"
+      id=" ${id}" pan_id=" ${id}" control_mode="standalone" parent_link="support" xyz=" 0.0 0.0 0.0"
+      ros_namespace="" />
     <gazebo reference="${name}_link">
       <turnGravityOff>true</turnGravityOff>

File: romea_rtls_transceiver_description/urdf/transceiver.xacro (robot description, xacro)
@@ -2,5 +2,5 @@
 <robot name="transceiver" xmlns:xacro="http://www.ros.org/wiki/xacro">
   <xacro:macro name="transceiver"
-    params="prefix name type conf id pan_id mode parent_link xyz ros_namespace">
+    params="prefix mode name type conf id pan_id control_mode parent_link xyz ros_namespace">
     <xacro:property name="file_conf"
       value="$(find romea_rtls_transceiver_description)/config/${type}_${conf}.yaml" />
@@ -39,21 +39,23 @@
       <child link="${link_name}" />
     </joint>
-    <gazebo>
-      <plugin name="driver" filename="libromea_gazebo_ros_rtls_transceiver.so">
-        <link_name>${link_name}</link_name>
-        <xyz>${xyz}</xyz>
-        <mode>${mode}</mode>
-        <transceiver_name>${name}</transceiver_name>
-        <transceiver_pan_id>${pan_id}</transceiver_pan_id>
-        <transceiver_id>${id}</transceiver_id>
-        <minimal_range>${minimal_range}</minimal_range>
-        <maximal_range>${maximal_range}</maximal_range>
-        <noise_a>${noise_a}</noise_a>
-        <noise_b>${noise_b}</noise_b>
-        <ros>
-          <namespace>${ros_namespace}</namespace>
-        </ros>
-      </plugin>
-    </gazebo>
+    <xacro:if value="${'simulation' in  mode}">
+      <gazebo>
+        <plugin name="driver" filename="libromea_gazebo_ros_rtls_transceiver.so">
+          <link_name>${link_name}</link_name>
+          <xyz>${xyz}</xyz>
+          <mode>${control_mode}</mode>
+          <transceiver_name>${name}</transceiver_name>
+          <transceiver_pan_id>${pan_id}</transceiver_pan_id>
+          <transceiver_id>${id}</transceiver_id>
+          <minimal_range>${minimal_range}</minimal_range>
+          <maximal_range>${maximal_range}</maximal_range>
+          <noise_a>${noise_a}</noise_a>
+          <noise_b>${noise_b}</noise_b>
+          <ros>
+            <namespace>${ros_namespace}</namespace>
+          </ros>
+        </plugin>
+      </gazebo>
+    </xacro:if>
   </xacro:macro>
 </robot>

Commit message: description: update xacro files
Signed-off-by: Jean Laneurit <jean.laneurit@inrae.fr>

File: romea_rtls_transceiver_description/urdf/anchor.xacro (robot description, xacro)
@@ -3,7 +3,7 @@
   <xacro:macro name="anchor" params="mode name type conf id pan_id">
     <xacro:include filename="$(find romea_rtls_transceiver_description)/urdf/transceiver.xacro" />
-    <link name="support" />
+    <link name="support_${name}"/>
     <xacro:transceiver prefix="" mode="${mode}" name="${name}" type="${type}" conf="${conf}"
-      id=" ${id}" pan_id=" ${id}" control_mode="standalone" parent_link="support" xyz=" 0.0 0.0 0.0"
+      id="${id}" pan_id="${pan_id}" control_mode="standalone" parent_link="support_${name}" xyz="0.0 0.0 0.0"
       ros_namespace="" />
     <gazebo reference="${name}_link">
